File: Sixnav.kicad_sch (KiCad schematic)
At the start: 33 parts, among them Q1 PT908-7C-F, Q2 PT908-7C-F, Q3 PT908-7C-F, Q4 PT908-7C-F, Q5 PT908-7C-F, Q6 PT908-7C-F, U1 Pico, U2 CD4051B

Commit message: Second Draft
It was only until after I finished routing this that I realized that the
PT908 and IR908 have flipped pin numbers. I'm going to have to aquire a
separate foorprint for the PT908.
Parts:
- D1, D2, D3, D4, D5, D6: footprint LED_THT:LED_D3.0mm_IRGrey -> SamacSys_Parts:IR9087CF
- Q1, Q2, Q3, Q4, Q5, Q6: footprint LED_THT:LED_D3.0mm_IRBlack -> SamacSys_Parts:IR9087CF
Changed lines of the file:
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@@
       (effects (font (size 1.27 1.27)) (justify left))
     )
-    (property "Footprint" "LED_THT:LED_D3.0mm_IRBlack" (id 2) (at 208.28 101.6 0)
+    (property "Footprint" "SamacSys_Parts:IR9087CF" (id 2) (at 208.28 101.6 0)
       (effects (font (size 1.27 1.27)) hide)
     )
@@
     (property "Reference" "D1" (id 0) (at 173.99 49.53 0))
     (property "Value" "IR908-7C-F" (id 1) (at 173.99 59.69 90))
-    (property "Footprint" "LED_THT:LED_D3.0mm_IRGrey" (id 2) (at 173.99 52.07 0)
+    (property "Footprint" "SamacSys_Parts:IR9087CF" (id 2) (at 173.99 52.07 0)
       (effects (font (size 1.27 1.27)) hide)
     )
@@
     (property "Reference" "D6" (id 0) (at 223.52 49.53 0))
     (property "Value" "IR908-7C-F" (id 1) (at 223.52 59.69 90))
-    (property "Footprint" "LED_THT:LED_D3.0mm_IRGrey" (id 2) (at 223.52 52.07 0)
+    (property "Footprint" "SamacSys_Parts:IR9087CF" (id 2) (at 223.52 52.07 0)
       (effects (font (size 1.27 1.27)) hide)
     )
@@
     (property "Reference" "D3" (id 0) (at 194.31 49.53 0))
     (property "Value" "IR908-7C-F" (id 1) (at 194.31 59.69 90))
-    (property "Footprint" "LED_THT:LED_D3.0mm_IRGrey" (id 2) (at 194.31 52.07 0)
+    (property "Footprint" "SamacSys_Parts:IR9087CF" (id 2) (at 194.31 52.07 0)
       (effects (font (size 1.27 1.27)) hide)
     )
@@
       (effects (font (size 1.27 1.27)) (justify left))
     )
-    (property "Footprint" "LED_THT:LED_D3.0mm_IRBlack" (id 2) (at 231.14 101.6 0)
+    (property "Footprint" "SamacSys_Parts:IR9087CF" (id 2) (at 231.14 101.6 0)
       (effects (font (size 1.27 1.27)) hide)
     )
@@
       (effects (font (size 1.27 1.27)) (justify left))
     )
-    (property "Footprint" "LED_THT:LED_D3.0mm_IRBlack" (id 2) (at 219.71 101.6 0)
+    (property "Footprint" "SamacSys_Parts:IR9087CF" (id 2) (at 219.71 101.6 0)
       (effects (font (size 1.27 1.27)) hide)
     )
@@
     (property "Reference" "D2" (id 0) (at 182.88 49.53 0))
     (property "Value" "IR908-7C-F" (id 1) (at 182.88 59.69 90))
-    (property "Footprint" "LED_THT:LED_D3.0mm_IRGrey" (id 2) (at 182.88 52.07 0)
+    (property "Footprint" "SamacSys_Parts:IR9087CF" (id 2) (at 182.88 52.07 0)
       (effects (font (size 1.27 1.27)) hide)
     )
@@
       (effects (font (size 1.27 1.27)) (justify left))
     )
-    (property "Footprint" "LED_THT:LED_D3.0mm_IRBlack" (id 2) (at 184.15 101.6 0)
+    (property "Footprint" "SamacSys_Parts:IR9087CF" (id 2) (at 184.15 101.6 0)
       (effects (font (size 1.27 1.27)) hide)
     )
@@
     (property "Reference" "D5" (id 0) (at 214.63 49.53 0))
     (property "Value" "IR908-7C-F" (id 1) (at 214.63 59.69 90))
-    (property "Footprint" "LED_THT:LED_D3.0mm_IRGrey" (id 2) (at 214.63 52.07 0)
+    (property "Footprint" "SamacSys_Parts:IR9087CF" (id 2) (at 214.63 52.07 0)
       (effects (font (size 1.27 1.27)) hide)
     )
@@
       (effects (font (size 1.27 1.27)) (justify left))
     )
-    (property "Footprint" "LED_THT:LED_D3.0mm_IRBlack" (id 2) (at 172.72 101.6 0)
+    (property "Footprint" "SamacSys_Parts:IR9087CF" (id 2) (at 172.72 101.6 0)
       (effects (font (size 1.27 1.27)) hide)
     )
@@
     (property "Reference" "D4" (id 0) (at 203.2 49.53 0))
     (property "Value" "IR908-7C-F" (id 1) (at 203.2 59.69 90))
-    (property "Footprint" "LED_THT:LED_D3.0mm_IRGrey" (id 2) (at 203.2 52.07 0)
+    (property "Footprint" "SamacSys_Parts:IR9087CF" (id 2) (at 203.2 52.07 0)
       (effects (font (size 1.27 1.27)) hide)
     )
@@
       (effects (font (size 1.27 1.27)) (justify left))
     )
-    (property "Footprint" "LED_THT:LED_D3.0mm_IRBlack" (id 2) (at 196.85 101.6 0)
+    (property "Footprint" "SamacSys_Parts:IR9087CF" (id 2) (at 196.85 101.6 0)
       (effects (font (size 1.27 1.27)) hide)
     )
@@
     )
     (path "/16bbf5c8-17c2-45be-bdc8-a6da3a3cc8de"
-      (reference "D1") (unit 1) (value "IR908-7C-F") (footprint "LED_THT:LED_D3.0mm_IRGrey")
+      (reference "D1") (unit 1) (value "IR908-7C-F") (footprint "SamacSys_Parts:IR9087CF")
     )
     (path "/9dfd217e-63cb-4686-9672-dc2be29baf75"
-      (reference "D2") (unit 1) (value "IR908-7C-F") (footprint "LED_THT:LED_D3.0mm_IRGrey")
+      (reference "D2") (unit 1) (value "IR908-7C-F") (footprint "SamacSys_Parts:IR9087CF")
     )
     (path "/323ea8bd-b4c6-4763-9284-128d37f64ff8"
-      (reference "D3") (unit 1) (value "IR908-7C-F") (footprint "LED_THT:LED_D3.0mm_IRGrey")
+      (reference "D3") (unit 1) (value "IR908-7C-F") (footprint "SamacSys_Parts:IR9087CF")
     )
     (path "/ddd06a71-621d-4990-878b-20a5df71305d"
-      (reference "D4") (unit 1) (value "IR908-7C-F") (footprint "LED_THT:LED_D3.0mm_IRGrey")
+      (reference "D4") (unit 1) (value "IR908-7C-F") (footprint "SamacSys_Parts:IR9087CF")
     )
     (path "/b3fc1c67-9d34-4066-8707-221b1db4f1ce"
-      (reference "D5") (unit 1) (value "IR908-7C-F") (footprint "LED_THT:LED_D3.0mm_IRGrey")
+      (reference "D5") (unit 1) (value "IR908-7C-F") (footprint "SamacSys_Parts:IR9087CF")
     )
     (path "/22d76b13-94d2-4b00-88e4-6c2ae3839254"
-      (reference "D6") (unit 1) (value "IR908-7C-F") (footprint "LED_THT:LED_D3.0mm_IRGrey")
+      (reference "D6") (unit 1) (value "IR908-7C-F") (footprint "SamacSys_Parts:IR9087CF")
     )
     (path "/408106ba-1c7c-4e1d-918e-76d733bc36a7"
@@
     )
     (path "/c5705971-f806-4ec8-9496-b86f09a59609"
-      (reference "Q1") (unit 1) (value "PT908-7C-F") (footprint "LED_THT:LED_D3.0mm_IRBlack")
+      (reference "Q1") (unit 1) (value "PT908-7C-F") (footprint "SamacSys_Parts:IR9087CF")
     )
     (path "/ac0c0e22-2325-4828-bded-ceda6deb1149"
-      (reference "Q2") (unit 1) (value "PT908-7C-F") (footprint "LED_THT:LED_D3.0mm_IRBlack")
+      (reference "Q2") (unit 1) (value "PT908-7C-F") (footprint "SamacSys_Parts:IR9087CF")
     )
     (path "/ea04ad93-5492-40b7-87af-8b9459a4ed79"
-      (reference "Q3") (unit 1) (value "PT908-7C-F") (footprint "LED_THT:LED_D3.0mm_IRBlack")
+      (reference "Q3") (unit 1) (value "PT908-7C-F") (footprint "SamacSys_Parts:IR9087CF")
     )
     (path "/140371dc-adb1-4ecb-80e5-82fead571f52"
-      (reference "Q4") (unit 1) (value "PT908-7C-F") (footprint "LED_THT:LED_D3.0mm_IRBlack")
+      (reference "Q4") (unit 1) (value "PT908-7C-F") (footprint "SamacSys_Parts:IR9087CF")
     )
     (path "/7b4d8924-d704-41bd-98c9-e262eb0599b4"
-      (reference "Q5") (unit 1) (value "PT908-7C-F") (footprint "LED_THT:LED_D3.0mm_IRBlack")
+      (reference "Q5") (unit 1) (value "PT908-7C-F") (footprint "SamacSys_Parts:IR9087CF")
     )
     (path "/37f5795f-9be5-4e2f-be06-09a1e0aafe69"
-      (reference "Q6") (unit 1) (value "PT908-7C-F") (footprint "LED_THT:LED_D3.0mm_IRBlack")
+      (reference "Q6") (unit 1) (value "PT908-7C-F") (footprint "SamacSys_Parts:IR9087CF")
     )
     (path "/8ffdd3a4-6d48-4257-a9b0-df5a9714f70f"

Commit message: PT908 footprint
Parts:
- Q1, Q2, Q3, Q4, Q5, Q6: footprint SamacSys_Parts:IR9087CF -> SamacSys_Parts:ELPT9087C
Connections:
- net GND: now also U1.13 (GND), U1.18 (GND), U1.3 (GND), U1.33 (AGND), U1.8 (GND)
- no-connect marks 38 -> 33
Other:
- moved on the sheet: H1, H2, H3, H4, H5, H6, H7
