File: src/ecad/SixnavPrototype.kicad_pcb (KiCad board)
At the start: 2 copper layers, 66 x 114.3 mm, 35 parts, among them Q1 PT908-7C-F, Q2 PT908-7C-F, Q3 PT908-7C-F, Q4 PT908-7C-F, Q5 PT908-7C-F, Q6 PT908-7C-F, U1 Pico, U2 CD4051B

Commit message: Revision 0.2.0 ECAD
Parts:
- added H11: TouchSpring, LibSixnavPrototype:TouchSpring10mm, F.Cu at (159.0, 138.2)
- added H12: TouchSpring, LibSixnavPrototype:TouchSpring10mm, F.Cu at (139.7, 104.8)
- added H13: TouchSpring, LibSixnavPrototype:TouchSpring10mm, F.Cu at (120.4, 138.1)
Routing:
- net +3.3V: track 280.1 -> 259.8 mm, vias 0 -> 4
- net /MUX_X5_Q6: track 80.9 -> 92.7 mm, vias 0 -> 6
- net /MUX_X0_Q1: track 122.5 -> 131.9 mm, vias 0 -> 2
- net /MUX_X2_Q3: track 69.9 -> 64.4 mm, vias 0 -> 6
- net /MUX_X1_Q2: track 111.2 -> 112.5 mm, vias 2 -> 0
- net /MUX_X4_Q5: track 77.8 -> 78.9 mm, vias 0 -> 6
- net /MUX_X3_Q4: vias 0 -> 2
Other:
- outline, holes or cut-outs redrawn
- board text removed: "JLCJLCJLCJLC"
