File: src/ecad/SixnavPrototype.kicad_sch (KiCad schematic)
At the start: 33 parts, among them Q1 PT908-7C-F, Q2 PT908-7C-F, Q3 PT908-7C-F, Q4 PT908-7C-F, Q5 PT908-7C-F, Q6 PT908-7C-F, U1 Pico, U2 CD4051B

Commit message: Revision 0.2.0 ECAD
Parts:
- added H11, H12, H13: TouchSpring, LibSixnavPrototype:TouchSpring10mm, symbol LibSixnavPrototype:TouchSpring
Connections:
- net GND: now also H11.1 (WIDE), H11.2 (PIN), H12.1 (WIDE), H12.2 (PIN), H13.1 (WIDE), H13.2 (PIN)
Other:
- note added: "Touch Springs"
